Commit message: Arduio control compile sucess

File: description/ros2_control.xacro (robot description, xacro)
@@ -1,7 +1,14 @@
 <?xml version="1.0"?>
 <robot xmlns:xacro="http://www.ros.org/wiki/xacro">
-    <ros2_control name="GazeboSystem" type="system">
+    <ros2_control name="RealRobot" type="system">
         <hardware>
-            <plugin>gazebo_ros2_control/GazeboSystem</plugin>
+            <plugin>diffdrive_arduino/DiffDriveArduinoHardware</plugin>
+            <param name="left_wheel_name">left_front_wheel_joint</param>
+            <param name="right_wheel_name">right_front_wheel_joint</param>
+            <param name="loop_rate">30</param>
+            <param name="device">/dev/ttyUSB0</param>
+            <param name="baud_rate">57600</param>
+            <param name="timeout_ms">1000</param>
+            <param name="enc_counts_per_rev">2640</param>
         </hardware>
         <joint name="left_front_wheel_joint">
@@ -10,6 +17,6 @@
                 <param name="max">10</param>
             </command_interface>
+            <state_interface name="position"/>
             <state_interface name="velocity"/>
-            <state_interface name="position"/>
         </joint>
         <joint name="right_front_wheel_joint">
@@ -18,28 +25,7 @@
                 <param name="max">10</param>
             </command_interface>
+            <state_interface name="position"/>
             <state_interface name="velocity"/>
-            <state_interface name="position"/>
-        </joint>
-        <joint name="left_rear_wheel_joint">
-            <command_interface name="velocity">
-                <param name="min">-10</param>
-                <param name="max">10</param>
-            </command_interface>
-            <state_interface name="velocity"/>
-            <state_interface name="position"/>
-        </joint>
-        <joint name="right_rear_wheel_joint">
-            <command_interface name="velocity">
-                <param name="min">-10</param>
-                <param name="max">10</param>
-            </command_interface>
-            <state_interface name="velocity"/>
-            <state_interface name="position"/>
         </joint>
     </ros2_control>
-    <gazebo>
-        <plugin name="gazebo_ros2_control" filename="libgazebo_ros2_control.so">
-            <parameters>$(find mybot_2wd)/config/my_controllers.yaml</parameters>
-        </plugin>
-    </gazebo>
 </robot>
