Commit message: ros2_control working

File: description/robot.urdf.xacro (robot description, xacro)
@@ -2,5 +2,6 @@
 <robot xmlns:xacro="http://www.ros.org/wiki/xacro"  name="robot">
     <xacro:include filename="robot_core.xacro" />
-    <xacro:include filename="gazebo_control.xacro" />
+    <xacro:include filename="ros2_control.xacro" />
+    <!-- <xacro:include filename="gazebo_control.xacro" /> -->
     <xacro:include filename="lidar.xacro" />
 </robot>

File: description/robot_core.xacro (robot description, xacro)
@@ -2,66 +2,25 @@
 <robot xmlns:xacro="http://www.ros.org/wiki/xacro" >
     <xacro:include filename="inertial_macros.xacro"/>
-    <!-- materials -->
-    <material name="white">
-        <color rgba="1 1 1 1" />
-    </material>
-    <material name="orange">
-        <color rgba="1 0.3 0.1 1"/>
-    </material>
-    <material name="blue">
-        <color rgba="0.2 0.2 1 1"/>
-    </material>
-    <material name="black">
-        <color rgba="0 0 0 1"/>
-    </material>
-     <material name="red">
-        <color rgba="1 0 0 1"/>
-    </material>
-    <!-- PARAMETERS -->
-    <!-- robot size -->
-    <!-- length (x) = 0.60 m, width (y) = 0.40 m, height (z) = 0.40 m -->
-    <xacro:property name="robot_length" value="0.60"/>
-    <xacro:property name="robot_width"  value="0.40"/>
-    <xacro:property name="robot_height" value="0.30"/>
-    <!-- wheel -->
-    <xacro:property name="wheel_diameter" value="0.10"/>
-    <xacro:property name="wheel_radius" value="${wheel_diameter/2.0}"/>
-    <xacro:property name="wheel_thickness" value="0.04"/> <!-- cylinder length -->
-    <!-- clearance between wheel center and chassis bottom -->
-    <xacro:property name="chassis_clearance" value="-0.04"/>
-    <!-- computed chassis center z: bottom = wheel_radius + clearance ; center = bottom + half-height -->
-    <xacro:property name="chassis_center_z" value="${wheel_radius + chassis_clearance + (robot_height/2.0)}"/>
-    <!-- wheel positions (front/back along x, left/right along y) -->
-    <!-- place the wheel pairs near the front and rear within the 0.6 m length -->
-    <xacro:property name="wheel_x_front" value="0.18"/>
-    <xacro:property name="wheel_x_rear"  value="-0.18"/>
-    <!-- lateral wheel offset; place slightly inset from edge: half width - small margin -->
-    <xacro:property name="wheel_y_offset" value="${(robot_width/2.0) + 0.025}"/>
-    <!-- BASE LINK -->
+    <material name="white"><color rgba="1 1 1 1" /></material>
+    <material name="blue"><color rgba="0.2 0.2 1 1"/></material>
     <link name="base_link"/>
-    <!-- CHASSIS mounted on base_link with a fixed joint (chassis sits above wheels) -->
     <joint name="chassis_joint" type="fixed">
         <parent link="base_link"/>
         <child link="chassis"/>
-        <origin xyz="0 0 ${chassis_center_z}"/>
+        <origin xyz="0 0 0.16"/>
     </joint>
     <link name="chassis">
         <visual>
-            <!-- chassis centered at base_link XY, elevated in Z -->
-            <origin xyz="0 0 0" />
             <geometry>
-                <box size="${robot_length} ${robot_width} ${robot_height}"/>
+                <box size="0.6 0.4 0.3"/>
             </geometry>
             <material name="white"/>
         </visual>
         <collision>
-            <origin xyz="0 0 0" />
             <geometry>
-                <box size="${robot_length} ${robot_width} ${robot_height}"/>
+                <box size="0.6 0.4 0.3"/>
             </geometry>
         </collision>
-        <!-- inertial using your inertial macro (mass chosen small; adjust if needed) -->
-        <xacro:inertial_box mass="3.0" x="${robot_length}" y="${robot_width}" z="${robot_height}">
-            <!-- origin of inertial box relative to chassis link frame -->
+        <xacro:inertial_box mass="3.0" x="0.6" y="0.4" z="0.3">
             <origin xyz="0 0 0" rpy="0 0 0"/>
         </xacro:inertial_box>
@@ -70,29 +29,23 @@
         <material>Gazebo/White</material>
     </gazebo>
-    <!-- FOUR WHEELS (two on each side: front/rear) -->
-    <!-- LEFT FRONT WHEEL -->
     <joint name="left_front_wheel_joint" type="continuous">
         <parent link="base_link"/>
         <child link="left_front_wheel"/>
-        <!-- wheel center is at its (x,y,0) in base_link frame (wheel center on ground z=0) -->
-        <origin xyz="${wheel_x_front} ${wheel_y_offset} 0" rpy="-${pi/2} 0 0"/>
-        <!-- rotation axis: z-axis in this joint frame (keeps same convention as your original file) -->
+        <origin xyz="0.18 0.225 0" rpy="-1.5707 0 0"/>
         <axis xyz="0 0 1"/>
     </joint>
     <link name="left_front_wheel">
         <visual>
-            <origin xyz="0 0 0"/>
             <geometry>
-                <cylinder radius="${wheel_radius}" length="${wheel_thickness}"/>
+                <cylinder radius="0.05" length="0.04"/>
             </geometry>
             <material name="blue"/>
         </visual>
         <collision>
-            <origin xyz="0 0 0"/>
             <geometry>
-                <cylinder radius="${wheel_radius}" length="${wheel_thickness}"/>
+                <cylinder radius="0.05" length="0.04"/>
             </geometry>
         </collision>
-        <xacro:inertial_cylinder mass="0.2" length="${wheel_thickness}" radius="${wheel_radius}">
+        <xacro:inertial_cylinder mass="0.2" length="0.04" radius="0.05">
             <origin xyz="0 0 0" rpy="0 0 0"/>
         </xacro:inertial_cylinder>
@@ -101,26 +54,23 @@
         <material>Gazebo/Blue</material>
     </gazebo>
-    <!-- LEFT REAR WHEEL -->
     <joint name="left_rear_wheel_joint" type="continuous">
         <parent link="base_link"/>
         <child link="left_rear_wheel"/>
-        <origin xyz="${wheel_x_rear} ${wheel_y_offset} 0" rpy="-${pi/2} 0 0"/>
+        <origin xyz="-0.18 0.225 0" rpy="-1.5707 0 0"/>
         <axis xyz="0 0 1"/>
     </joint>
     <link name="left_rear_wheel">
         <visual>
-            <origin xyz="0 0 0"/>
             <geometry>
-                <cylinder radius="${wheel_radius}" length="${wheel_thickness}"/>
+                <cylinder radius="0.05" length="0.04"/>
             </geometry>
             <material name="blue"/>
         </visual>
         <collision>
-            <origin xyz="0 0 0"/>
             <geometry>
-                <cylinder radius="${wheel_radius}" length="${wheel_thickness}"/>
+                <cylinder radius="0.05" length="0.04"/>
             </geometry>
         </collision>
-        <xacro:inertial_cylinder mass="0.2" length="${wheel_thickness}" radius="${wheel_radius}">
+        <xacro:inertial_cylinder mass="0.2" length="0.04" radius="0.05">
             <origin xyz="0 0 0" rpy="0 0 0"/>
         </xacro:inertial_cylinder>
@@ -128,28 +78,26 @@
     <gazebo reference="left_rear_wheel">
         <material>Gazebo/Blue</material>
+        <mu1 value="0.001"/>
+        <mu2 value="0.001"/>
     </gazebo>
-    <!-- RIGHT FRONT WHEEL -->
     <joint name="right_front_wheel_joint" type="continuous">
         <parent link="base_link"/>
         <child link="right_front_wheel"/>
-        <origin xyz="${wheel_x_front} -${wheel_y_offset} 0" rpy="${pi/2} 0 0"/>
-        <!-- axis inverted to keep consistent rotation direction like your original right wheel -->
+        <origin xyz="0.18 -0.225 0" rpy="1.5707 0 0"/>
         <axis xyz="0 0 -1"/>
     </joint>
     <link name="right_front_wheel">
         <visual>
-            <origin xyz="0 0 0"/>
             <geometry>
-                <cylinder radius="${wheel_radius}" length="${wheel_thickness}"/>
+                <cylinder radius="0.05" length="0.04"/>
             </geometry>
             <material name="blue"/>
         </visual>
         <collision>
-            <origin xyz="0 0 0"/>
             <geometry>
-                <cylinder radius="${wheel_radius}" length="${wheel_thickness}"/>
+                <cylinder radius="0.05" length="0.04"/>
             </geometry>
         </collision>
-        <xacro:inertial_cylinder mass="0.2" length="${wheel_thickness}" radius="${wheel_radius}">
+        <xacro:inertial_cylinder mass="0.2" length="0.04" radius="0.05">
             <origin xyz="0 0 0" rpy="0 0 0"/>
         </xacro:inertial_cylinder>
@@ -158,26 +106,23 @@
         <material>Gazebo/Blue</material>
     </gazebo>
-    <!-- RIGHT REAR WHEEL -->
     <joint name="right_rear_wheel_joint" type="continuous">
         <parent link="base_link"/>
         <child link="right_rear_wheel"/>
-        <origin xyz="${wheel_x_rear} -${wheel_y_offset} 0" rpy="${pi/2} 0 0"/>
+        <origin xyz="-0.18 -0.225 0" rpy="1.5707 0 0"/>
         <axis xyz="0 0 -1"/>
     </joint>
     <link name="right_rear_wheel">
         <visual>
-            <origin xyz="0 0 0"/>
             <geometry>
-                <cylinder radius="${wheel_radius}" length="${wheel_thickness}"/>
+                <cylinder radius="0.05" length="0.04"/>
             </geometry>
             <material name="blue"/>
         </visual>
         <collision>
-            <origin xyz="0 0 0"/>
             <geometry>
-                <cylinder radius="${wheel_radius}" length="${wheel_thickness}"/>
+                <cylinder radius="0.05" length="0.04"/>
             </geometry>
         </collision>
-        <xacro:inertial_cylinder mass="0.2" length="${wheel_thickness}" radius="${wheel_radius}">
+        <xacro:inertial_cylinder mass="0.2" length="0.04" radius="0.05">
             <origin xyz="0 0 0" rpy="0 0 0"/>
         </xacro:inertial_cylinder>
@@ -185,4 +130,6 @@
     <gazebo reference="right_rear_wheel">
         <material>Gazebo/Blue</material>
+        <mu1 value="0.001"/>
+        <mu2 value="0.001"/>
     </gazebo>
 </robot>

Commit message: Break Gazebo Sim

File: description/robot.urdf.xacro (robot description, xacro)
@@ -1,4 +1,5 @@
 <?xml version="1.0"?>
 <robot xmlns:xacro="http://www.ros.org/wiki/xacro"  name="robot">
+    <xacro:arg name="sim_mode" default="false"/>
     <xacro:include filename="robot_core.xacro" />
     <xacro:include filename="ros2_control.xacro" />

File: description/ros2_control.xacro (robot description, xacro)
@@ -1,31 +1,62 @@
 <?xml version="1.0"?>
 <robot xmlns:xacro="http://www.ros.org/wiki/xacro">
-    <ros2_control name="RealRobot" type="system">
-        <hardware>
-            <plugin>diffdrive_arduino/DiffDriveArduinoHardware</plugin>
-            <param name="left_wheel_name">left_front_wheel_joint</param>
-            <param name="right_wheel_name">right_front_wheel_joint</param>
-            <param name="loop_rate">30</param>
-            <param name="device">/dev/ttyUSB0</param>
-            <param name="baud_rate">57600</param>
-            <param name="timeout_ms">1000</param>
-            <param name="enc_counts_per_rev">2515</param>
-        </hardware>
-        <joint name="left_front_wheel_joint">
-            <command_interface name="velocity">
-                <param name="min">-10</param>
-                <param name="max">10</param>
-            </command_interface>
-            <state_interface name="position"/>
-            <state_interface name="velocity"/>
-        </joint>
-        <joint name="right_front_wheel_joint">
-            <command_interface name="velocity">
-                <param name="min">-10</param>
-                <param name="max">10</param>
-            </command_interface>
-            <state_interface name="position"/>
-            <state_interface name="velocity"/>
-        </joint>
-    </ros2_control>
+    <xacro:unless value="$(arg sim_mode)">
+        <ros2_control name="RealRobot" type="system">
+            <hardware>
+                <plugin>diffdrive_arduino/DiffDriveArduinoHardware</plugin>
+                <param name="left_wheel_name">left_front_wheel_joint</param>
+                <param name="right_wheel_name">right_front_wheel_joint</param>
+                <param name="loop_rate">30</param>
+                <param name="device">/dev/ttyUSB0</param>
+                <param name="baud_rate">57600</param>
+                <param name="timeout_ms">1000</param>
+                <param name="enc_counts_per_rev">2515</param>
+            </hardware>
+            <joint name="left_front_wheel_joint">
+                <command_interface name="velocity">
+                    <param name="min">-10</param>
+                    <param name="max">10</param>
+                </command_interface>
+                <state_interface name="position"/>
+                <state_interface name="velocity"/>
+            </joint>
+            <joint name="right_front_wheel_joint">
+                <command_interface name="velocity">
+                    <param name="min">-10</param>
+                    <param name="max">10</param>
+                </command_interface>
+                <state_interface name="position"/>
+                <state_interface name="velocity"/>
+            </joint>
+        </ros2_control>
+    </xacro:unless>
+    <xacro:if value="$(arg sim_mode)">
+        <ros2_control name="GazeboSystem" type="system">
+            <hardware>
+                <plugin>gazebo_ros2_control/GazeboSystem</plugin>
+            </hardware>
+            <joint name="left_front_wheel_joint">
+                <command_interface name="velocity">
+                    <param name="min">-10</param>
+                    <param name="max">10</param>
+                </command_interface>
+                <state_interface name="velocity"/>
+                <state_interface name="position"/>
+            </joint>
+            <joint name="right_front_wheel_joint">
+                <command_interface name="velocity">
+                    <param name="min">-10</param>
+                    <param name="max">10</param>
+                </command_interface>
+                <state_interface name="velocity"/>
+                <state_interface name="position"/>
+            </joint>
+        </ros2_control>
+    </xacro:if>
+    <gazebo>
+        <plugin name="gazebo_ros2_control" filename="libgazebo_ros2_control.so">
+            <parameters>$(find mybot_2wd)/config/my_controllers.yaml</parameters>
+            <parameters>$(find mybot_2wd)/config/gaz_ros2_ctl_use_sim.yaml</parameters>
+        </plugin>
+    </gazebo>
 </robot>
