Commit message: ros2_control working Laser scan TF messed

File: description/robot_core.xacro (robot description, xacro)
@@ -78,6 +78,4 @@
     <gazebo reference="left_rear_wheel">
         <material>Gazebo/Blue</material>
-        <mu1 value="0.001"/>
-        <mu2 value="0.001"/>
     </gazebo>
     <joint name="right_front_wheel_joint" type="continuous">
@@ -130,6 +128,4 @@
     <gazebo reference="right_rear_wheel">
         <material>Gazebo/Blue</material>
-        <mu1 value="0.001"/>
-        <mu2 value="0.001"/>
     </gazebo>
 </robot>

File: description/ros2_control.xacro (robot description, xacro)
@@ -21,4 +21,20 @@
             <state_interface name="position"/>
         </joint>
+        <joint name="left_rear_wheel_joint">
+            <command_interface name="velocity">
+                <param name="min">-10</param>
+                <param name="max">10</param>
+            </command_interface>
+            <state_interface name="velocity"/>
+            <state_interface name="position"/>
+        </joint>
+        <joint name="right_rear_wheel_joint">
+            <command_interface name="velocity">
+                <param name="min">-10</param>
+                <param name="max">10</param>
+            </command_interface>
+            <state_interface name="velocity"/>
+            <state_interface name="position"/>
+        </joint>
     </ros2_control>
     <gazebo>

Commit message: Rviz laser scan rotation fixed

File: description/robot_core.xacro (robot description, xacro)
@@ -59,4 +59,5 @@
         <origin xyz="-0.18 0.225 0" rpy="-1.5707 0 0"/>
         <axis xyz="0 0 1"/>
+        <!-- <mimic joint="left_front_wheel_joint" multiplier="1.0" /> -->
     </joint>
     <link name="left_rear_wheel">
@@ -78,4 +79,6 @@
     <gazebo reference="left_rear_wheel">
         <material>Gazebo/Blue</material>
+        <mu1 value="0.001"/>
+        <mu2 value="0.001"/>
     </gazebo>
     <joint name="right_front_wheel_joint" type="continuous">
@@ -109,4 +112,5 @@
         <origin xyz="-0.18 -0.225 0" rpy="1.5707 0 0"/>
         <axis xyz="0 0 -1"/>
+        <!-- <mimic joint="right_front_wheel_joint" multiplier="1.0" /> -->
     </joint>
     <link name="right_rear_wheel">
@@ -128,4 +132,6 @@
     <gazebo reference="right_rear_wheel">
         <material>Gazebo/Blue</material>
+        <mu1 value="0.001"/>
+        <mu2 value="0.001"/>
     </gazebo>
 </robot>

Commit message: Basic SLAM

File: description/robot_core.xacro (robot description, xacro)
@@ -4,5 +4,14 @@
     <material name="white"><color rgba="1 1 1 1" /></material>
     <material name="blue"><color rgba="0.2 0.2 1 1"/></material>
+    <!-- BASE LINK -->
     <link name="base_link"/>
+    <!-- BASE_FOOTPRINT LINK -->
+    <joint name="base_footprint_joint" type="fixed">
+        <parent link="base_link"/>
+        <child link="base_footprint"/>
+        <origin xyz="0 0 0" rpy="0 0 0"/>
+    </joint>
+    <link name="base_footprint">
+    </link>
     <joint name="chassis_joint" type="fixed">
         <parent link="base_link"/>
@@ -13,5 +22,5 @@
         <visual>
             <geometry>
-                <box size="0.6 0.4 0.3"/>
+                <box size="0.6 0.44 0.3"/>
             </geometry>
             <material name="white"/>
@@ -19,8 +28,8 @@
         <collision>
             <geometry>
-                <box size="0.6 0.4 0.3"/>
+                <box size="0.6 0.44 0.3"/>
             </geometry>
         </collision>
-        <xacro:inertial_box mass="3.0" x="0.6" y="0.4" z="0.3">
+        <xacro:inertial_box mass="3.0" x="0.6" y="0.44" z="0.3">
             <origin xyz="0 0 0" rpy="0 0 0"/>
         </xacro:inertial_box>
@@ -32,5 +41,5 @@
         <parent link="base_link"/>
         <child link="left_front_wheel"/>
-        <origin xyz="0.18 0.225 0" rpy="-1.5707 0 0"/>
+        <origin xyz="0.18 0.275 0" rpy="-1.5707 0 0"/>
         <axis xyz="0 0 1"/>
     </joint>
@@ -57,5 +66,5 @@
         <parent link="base_link"/>
         <child link="left_rear_wheel"/>
-        <origin xyz="-0.18 0.225 0" rpy="-1.5707 0 0"/>
+        <origin xyz="-0.18 0.275 0" rpy="-1.5707 0 0"/>
         <axis xyz="0 0 1"/>
         <!-- <mimic joint="left_front_wheel_joint" multiplier="1.0" /> -->
@@ -85,5 +94,5 @@
         <parent link="base_link"/>
         <child link="right_front_wheel"/>
-        <origin xyz="0.18 -0.225 0" rpy="1.5707 0 0"/>
+        <origin xyz="0.18 -0.275 0" rpy="1.5707 0 0"/>
         <axis xyz="0 0 -1"/>
     </joint>
@@ -110,5 +119,5 @@
         <parent link="base_link"/>
         <child link="right_rear_wheel"/>
-        <origin xyz="-0.18 -0.225 0" rpy="1.5707 0 0"/>
+        <origin xyz="-0.18 -0.275 0" rpy="1.5707 0 0"/>
         <axis xyz="0 0 -1"/>
         <!-- <mimic joint="right_front_wheel_joint" multiplier="1.0" /> -->
