Commit message: IMU Bench test and IMU in URDF

File: description/lidar.xacro (robot description, xacro)
@@ -4,6 +4,7 @@
     <parent link="chassis"/>
     <child link="laser_frame"/>
-    <origin xyz="0 0 0.17" rpy="0 0 0"/>
+    <origin xyz="-0.07 0 0.17" rpy="0 0 0"/>
     </joint>
+    <material name="red"><color rgba="1.0 0 0 1.0"/></material>
     <link name="laser_frame">
         <visual>

File: description/robot.urdf.xacro (robot description, xacro)
@@ -6,3 +6,4 @@
     <!-- <xacro:include filename="gazebo_control.xacro" /> -->
     <xacro:include filename="lidar.xacro" />
+    <xacro:include filename="imu.xacro"/>
 </robot>
