Commit message: Depth cam failed

File: description/depth_camera.xacro (robot description, xacro)
@@ -5,5 +5,5 @@
     <parent link="chassis"/>
     <child link="camera_link"/>
-    <origin xyz="0.05 0 0.27" rpy="0 0.11 0"/>
+    <origin xyz="0.05 0 0.1175" rpy="0 0.11 0"/>
   </joint>
   <!-- ================= MIRRORED FRAME (HACK) ================= -->
