Commit message: Upgraded Files for Gazebo Ignition

File: description/camera.xacro (robot description, xacro)
@@ -4,5 +4,11 @@
         <parent link="chassis"/>
         <child link="camera_link"/>
-        <origin xyz="0.05 0 0.27" rpy="0 0 0"/>
+        <origin xyz="0.05 0 0.27" rpy="0 0.11 0"/>
+    </joint>
+    <link name="mybot_2wd/base_link/camera"/>
+        <joint name="gazebo_camera_tf_joint" type="fixed">
+        <parent link="camera_link"/>
+        <child link="mybot_2wd/base_link/camera"/>
+        <origin xyz="0 0 0" rpy="0 0 0"/>
     </joint>
     <link name="camera_link">
@@ -27,4 +33,5 @@
             <update_rate>10</update_rate>
             <camera>
+                <camera_info_topic>camera/camera_info</camera_info_topic>
                 <horizontal_fov>1.047</horizontal_fov>
                 <image>
@@ -38,7 +45,6 @@
                 </clip>
             </camera>
-            <plugin name="camera_controller" filename="libgazebo_ros_camera.so">
-                <frame_name>camera_link_optical</frame_name>
-            </plugin>
+            <topic>camera/image_raw</topic>
+            <gz_frame_id>camera_link_optical</gz_frame_id>
         </sensor>
     </gazebo>

File: description/lidar.xacro (robot description, xacro)
@@ -5,4 +5,11 @@
     <child link="laser_frame"/>
     <origin xyz="-0.07 0 0.17" rpy="0 0 0"/>
+    </joint>
+    <!-- Gazebo-generated lidar frame -->
+    <link name="mybot_2wd/base_link/laser"/>
+    <joint name="gazebo_laser_tf_joint" type="fixed">
+    <parent link="laser_frame"/>
+    <child link="mybot_2wd/base_link/laser"/>
+    <origin xyz="0 0 0" rpy="0 0 0"/>
     </joint>
     <material name="red"><color rgba="1.0 0 0 1.0"/></material>
@@ -25,9 +32,10 @@
     <gazebo reference="laser_frame">
         <material>Gazebo/Red</material>
-        <sensor name="laser" type="ray">
+        <sensor name="laser" type="gpu_lidar">
             <pose> 0 0 0 0 0 0 </pose>
-            <visualize>false</visualize>
+            <visualize>true</visualize>
             <update_rate>10</update_rate>
-            <ray>
+            <ignition_frame_id>laser_frame</ignition_frame_id>
+            <lidar>
                 <scan>
                     <horizontal>
@@ -43,12 +51,7 @@
                     <resolution>0.01</resolution>
                 </range>
-            </ray>
-            <plugin name="laser_controller" filename="libgazebo_ros_ray_sensor.so">
-                <ros>
-                    <argument>~/out:=scan</argument>
-                </ros>
-                <output_type>sensor_msgs/LaserScan</output_type>
-                <frame_name>laser_frame</frame_name>
-            </plugin>
+            </lidar>
+            <topic>scan</topic>
+            <!-- <frame_id>laser_frame</frame_id> -->
         </sensor>
     </gazebo>

File: description/robot.urdf.xacro (robot description, xacro)
@@ -5,6 +5,6 @@
     <xacro:include filename="ros2_control.xacro" />
     <!-- <xacro:include filename="gazebo_control.xacro" /> -->
-    <!-- <xacro:include filename="camera.xacro" /> -->
-    <xacro:include filename="depth_camera.xacro" />
+    <xacro:include filename="camera.xacro" />
+    <!-- <xacro:include filename="depth_camera.xacro" /> -->
     <xacro:include filename="lidar.xacro" />
     <xacro:include filename="imu.xacro"/>

File: description/ros2_control.xacro (robot description, xacro)
@@ -34,5 +34,5 @@
         <ros2_control name="GazeboSystem" type="system">
             <hardware>
-                <plugin>gazebo_ros2_control/GazeboSystem</plugin>
+                <plugin>gz_ros2_control/GazeboSimSystem</plugin>
             </hardware>
             <joint name="left_front_wheel_joint">
@@ -55,5 +55,5 @@
     </xacro:if>
     <gazebo>
-        <plugin name="gazebo_ros2_control" filename="libgazebo_ros2_control.so">
+        <plugin name="gz_ros2_control::GazeboSimROS2ControlPlugin" filename="libgz_ros2_control-system.so">
             <parameters>$(find mybot_2wd)/config/my_controllers.yaml</parameters>
             <parameters>$(find mybot_2wd)/config/gaz_ros2_ctl_use_sim.yaml</parameters>

Commit message: Ball tracker successful

File: description/camera.xacro (robot description, xacro)
@@ -4,5 +4,5 @@
         <parent link="chassis"/>
         <child link="camera_link"/>
-        <origin xyz="0.05 0 0.27" rpy="0 0.11 0"/>
+        <origin xyz="0.05 0 0.1175" rpy="0 0.42 0"/>
     </joint>
     <link name="mybot_2wd/base_link/camera"/>

File: description/lidar.xacro (robot description, xacro)
@@ -4,5 +4,5 @@
     <parent link="chassis"/>
     <child link="laser_frame"/>
-    <origin xyz="-0.07 0 0.17" rpy="0 0 0"/>
+    <origin xyz="-0.04 0 0.1825" rpy="0 0 0"/>
     </joint>
     <!-- Gazebo-generated lidar frame -->

File: description/robot_core.xacro (robot description, xacro)
@@ -17,10 +17,10 @@
         <parent link="base_link"/>
         <child link="chassis"/>
-        <origin xyz="0 0 0.16"/>
+        <origin xyz="0 0 0.167"/>
     </joint>
     <link name="chassis">
         <visual>
             <geometry>
-                <box size="0.6 0.44 0.3"/>
+                <box size="0.6 0.44 0.265"/>
             </geometry>
             <material name="white"/>
@@ -28,8 +28,8 @@
         <collision>
             <geometry>
-                <box size="0.6 0.44 0.3"/>
+                <box size="0.6 0.44 0.265"/>
             </geometry>
         </collision>
-        <xacro:inertial_box mass="3.0" x="0.6" y="0.44" z="0.3">
+        <xacro:inertial_box mass="3.0" x="0.6" y="0.44" z="0.265">
             <origin xyz="0 0 0" rpy="0 0 0"/>
         </xacro:inertial_box>
@@ -47,5 +47,5 @@
         <visual>
             <geometry>
-                <cylinder radius="0.05" length="0.04"/>
+                <cylinder radius="0.0525" length="0.04"/>
             </geometry>
             <material name="blue"/>
@@ -53,8 +53,8 @@
         <collision>
             <geometry>
-                <cylinder radius="0.05" length="0.04"/>
+                <cylinder radius="0.0525" length="0.04"/>
             </geometry>
         </collision>
-        <xacro:inertial_cylinder mass="0.2" length="0.04" radius="0.05">
+        <xacro:inertial_cylinder mass="0.2" length="0.04" radius="0.0525">
             <origin xyz="0 0 0" rpy="0 0 0"/>
         </xacro:inertial_cylinder>
@@ -73,5 +73,5 @@
         <visual>
             <geometry>
-                <cylinder radius="0.05" length="0.04"/>
+                <cylinder radius="0.0525" length="0.04"/>
             </geometry>
             <material name="blue"/>
@@ -79,8 +79,8 @@
         <collision>
             <geometry>
-                <cylinder radius="0.05" length="0.04"/>
+                <cylinder radius="0.0525" length="0.04"/>
             </geometry>
         </collision>
-        <xacro:inertial_cylinder mass="0.2" length="0.04" radius="0.05">
+        <xacro:inertial_cylinder mass="0.2" length="0.04" radius="0.0525">
             <origin xyz="0 0 0" rpy="0 0 0"/>
         </xacro:inertial_cylinder>
@@ -100,5 +100,5 @@
         <visual>
             <geometry>
-                <cylinder radius="0.05" length="0.04"/>
+                <cylinder radius="0.0525" length="0.04"/>
             </geometry>
             <material name="blue"/>
@@ -106,8 +106,8 @@
         <collision>
             <geometry>
-                <cylinder radius="0.05" length="0.04"/>
+                <cylinder radius="0.0525" length="0.04"/>
             </geometry>
         </collision>
-        <xacro:inertial_cylinder mass="0.2" length="0.04" radius="0.05">
+        <xacro:inertial_cylinder mass="0.2" length="0.04" radius="0.0525">
             <origin xyz="0 0 0" rpy="0 0 0"/>
         </xacro:inertial_cylinder>
@@ -126,5 +126,5 @@
         <visual>
             <geometry>
-                <cylinder radius="0.05" length="0.04"/>
+                <cylinder radius="0.0525" length="0.04"/>
             </geometry>
             <material name="blue"/>
@@ -132,8 +132,8 @@
         <collision>
             <geometry>
-                <cylinder radius="0.05" length="0.04"/>
+                <cylinder radius="0.0525" length="0.04"/>
             </geometry>
         </collision>
-        <xacro:inertial_cylinder mass="0.2" length="0.04" radius="0.05">
+        <xacro:inertial_cylinder mass="0.2" length="0.04" radius="0.0525">
             <origin xyz="0 0 0" rpy="0 0 0"/>
         </xacro:inertial_cylinder>

Commit message: Added Camera for April Tag Nav

File: description/camera.xacro (robot description, xacro)
@@ -1,45 +1,50 @@
 <?xml version="1.0"?>
-<robot xmlns:xacro="http://www.ros.org/wiki/xacro" >
-    <joint name="camera_joint" type="fixed">
-        <parent link="chassis"/>
-        <child link="camera_link"/>
-        <origin xyz="0.05 0 0.27" rpy="0 0 0"/>
-    </joint>
-    <link name="camera_link">
-        <visual>
-            <geometry>
-                <box size="0.03 0.07 0.035"/>
-            </geometry>
-            <material name="red"/>
-        </visual>
-    </link>
-    <joint name="camera_optical_joint" type="fixed">
-        <parent link="camera_link"/>
-        <child link="camera_link_optical"/>
-        <origin xyz="0 0 0" rpy="${-pi/2} 0 ${-pi/2}"/>
-    </joint>
-    <link name="camera_link_optical"></link>
-    <gazebo reference="camera_link">
-        <material>Gazebo/Red</material>
-        <sensor name="camera" type="camera">
-            <pose> 0 0 0 0 0 0 </pose>
-            <visualize>true</visualize>
-            <update_rate>10</update_rate>
-            <camera>
-                <horizontal_fov>1.047</horizontal_fov>
-                <image>
-                    <format>R8G8B8</format>
-                    <width>640</width>
-                    <height>480</height>
-                </image>
-                <clip>
-                    <near>0.1</near>
-                    <far>10.0</far>
-                </clip>
-            </camera>
-            <plugin name="camera_controller" filename="libgazebo_ros_camera.so">
-                <frame_name>camera_link_optical</frame_name>
-            </plugin>
-        </sensor>
-    </gazebo>
+<robot xmlns:xacro="http://www.ros.org/wiki/xacro">
+  <!-- Camera mounting with upward tilt for wall-mounted tags (50-100cm height) -->
+  <joint name="camera_joint" type="fixed">
+    <parent link="chassis"/>
+    <child link="camera_link"/>
+    <!-- Tilt camera slightly upward (0.15 rad ≈ 8.6°) to see wall-mounted tags better -->
+    <origin xyz="0.05 0 0.27" rpy="0 0.15 0"/>
+  </joint>
+  <link name="camera_link">
+    <visual>
+      <geometry>
+        <box size="0.03 0.07 0.035"/>
+      </geometry>
+      <material name="red"/>
+    </visual>
+  </link>
+  <!-- Optical frame (IMPORTANT for AprilTag) -->
+  <joint name="camera_optical_joint" type="fixed">
+    <parent link="camera_link"/>
+    <child link="camera_link_optical"/>
+    <!-- ROS optical frame convention -->
+    <origin xyz="0 0 0" rpy="-1.5708 0 -1.5708"/>
+  </joint>
+  <link name="camera_link_optical"/>
+  <!-- Gazebo camera sensor -->
+  <gazebo reference="camera_link">
+    <sensor name="camera" type="camera">
+      <pose>0 0 0 0 0 0</pose>
+      <visualize>true</visualize>
+      <update_rate>30</update_rate>
+      <camera>
+        <horizontal_fov>1.047</horizontal_fov>
+        <image>
+          <width>640</width>
+          <height>480</height>
+          <format>R8G8B8</format>
+        </image>
+        <clip>
+          <near>0.1</near>
+          <far>10.0</far>
+        </clip>
+      </camera>
+      <plugin name="camera_controller" filename="libgazebo_ros_camera.so">
+        <camera_name>camera</camera_name>
+        <frame_name>camera_link_optical</frame_name>
+      </plugin>
+    </sensor>
+  </gazebo>
 </robot>

Commit message: Camera Alignemnt added

File: description/camera.xacro (robot description, xacro)
@@ -4,5 +4,5 @@
         <parent link="chassis"/>
         <child link="camera_link"/>
-        <origin xyz="0.05 0 0.1175" rpy="0 0.42 0"/>
+        <origin xyz="0.125 0.155 0.145" rpy="0 0.15 0"/>
     </joint>
     <link name="mybot_2wd/base_link/camera"/>
